File: kicad/mycropad.sch (KiCad schematic (older format))
At the start: 29 parts, among them SW1 SW_Push, SW2 SW_Push, SW3 SW_Push, SW4 SW_Push, SW5 SW_Push, SW6 SW_Push, SW7 SW_Push, SW8 SW_Push, U1 Pico, U2 SN74AHCT125N

Commit message: Updated footprints for SK6812 MINI-E.
Parts:
- C1, C2, C3, C4, C5, C6, C7, C8, D1: LCSC (none) -> C13585
Changed lines of the file:
@@
 F 2 "mycropad:LED_SK6812MINI-E_REV02_PLCC4_3.5x3.5mm_P1.75mm" H 8050 1100 50  0001 L TNN
 F 3 "https://cdn-shop.adafruit.com/product-files/4960/4960_SK6812MINI-E_REV02_EN.pdf" H 8100 1025 50  0001 L TNN
+F 4 "C13585" H 8000 1400 50  0001 C CNN "LCSC"
 	1    8000 1400
 	1    0    0    -1
@@
 F 2 "Capacitor_SMD:C_1206_3216Metric_Pad1.33x1.80mm_HandSolder" H 8288 850 50  0001 C CNN
 F 3 "~" H 8250 1000 50  0001 C CNN
+F 4 "C13585" H 8250 1000 50  0001 C CNN "LCSC"
 	1    8250 1000
 	0    1    1    0
@@
 F 2 "Capacitor_SMD:C_1206_3216Metric_Pad1.33x1.80mm_HandSolder" H 9238 850 50  0001 C CNN
 F 3 "~" H 9200 1000 50  0001 C CNN
+F 4 "C13585" H 9200 1000 50  0001 C CNN "LCSC"
 	1    9200 1000
 	0    1    1    0
@@
 F 2 "Capacitor_SMD:C_1206_3216Metric_Pad1.33x1.80mm_HandSolder" H 10188 850 50  0001 C CNN
 F 3 "~" H 10150 1000 50  0001 C CNN
+F 4 "C13585" H 10150 1000 50  0001 C CNN "LCSC"
 	1    10150 1000
 	0    1    1    0
@@
 F 2 "Capacitor_SMD:C_1206_3216Metric_Pad1.33x1.80mm_HandSolder" H 8288 2200 50  0001 C CNN
 F 3 "~" H 8250 2350 50  0001 C CNN
+F 4 "C13585" H 8250 2350 50  0001 C CNN "LCSC"
 	1    8250 2350
 	0    1    1    0
@@
 F 2 "Capacitor_SMD:C_1206_3216Metric_Pad1.33x1.80mm_HandSolder" H 9238 2200 50  0001 C CNN
 F 3 "~" H 9200 2350 50  0001 C CNN
+F 4 "C13585" H 9200 2350 50  0001 C CNN "LCSC"
 	1    9200 2350
 	0    1    1    0
@@
 F 2 "Capacitor_SMD:C_1206_3216Metric_Pad1.33x1.80mm_HandSolder" H 10188 2200 50  0001 C CNN
 F 3 "~" H 10150 2350 50  0001 C CNN
+F 4 "C13585" H 10150 2350 50  0001 C CNN "LCSC"
 	1    10150 2350
 	0    1    1    0
@@
 F 2 "Capacitor_SMD:C_1206_3216Metric_Pad1.33x1.80mm_HandSolder" H 8288 3550 50  0001 C CNN
 F 3 "~" H 8250 3700 50  0001 C CNN
+F 4 "C13585" H 8250 3700 50  0001 C CNN "LCSC"
 	1    8250 3700
 	0    1    1    0
@@
 F 2 "Capacitor_SMD:C_1206_3216Metric_Pad1.33x1.80mm_HandSolder" H 9238 3550 50  0001 C CNN
 F 3 "~" H 9200 3700 50  0001 C CNN
+F 4 "C13585" H 9200 3700 50  0001 C CNN "LCSC"
 	1    9200 3700
 	0    1    1    0

Commit message: mycropad v0.2 started.
Parts:
- D1, D2, D3, D4, D5, D6, D7, D8: footprint mycropad:LED_SK6812MINI-E_REV02_PLCC4_3.5x3.5mm_P1.75mm -> mycropad:LED_SK6812MINI-E_REV02_PLCC4_3.5x3.5mm_P1.75mm___V2
Other:
- note removed: "Mycropad board"
Changed lines of the file:
@@
 encoding utf-8
 Sheet 1 1
-Title ""
-Date ""
-Rev ""
-Comp ""
+Title "Mycropad Board"
+Date "2021-11-11"
+Rev "v0.2"
+Comp "meronz"
 Comment1 ""
 Comment2 ""
@@
 Text Notes 2850 4050 2    50   ~ 0
 Raspberry PI
-Text Notes 7400 7500 0    50   ~ 0
-Mycropad board
 $Comp
 L power:GND #PWR0137
@@
 F 0 "D1" H 8250 1300 50  0000 L CNN
 F 1 "SK6812MINI-E" H 8344 1355 50  0001 L CNN
-F 2 "mycropad:LED_SK6812MINI-E_REV02_PLCC4_3.5x3.5mm_P1.75mm" H 8050 1100 50  0001 L TNN
+F 2 "mycropad:LED_SK6812MINI-E_REV02_PLCC4_3.5x3.5mm_P1.75mm___V2" H 8050 1100 50  0001 L TNN
 F 3 "https://cdn-shop.adafruit.com/product-files/4960/4960_SK6812MINI-E_REV02_EN.pdf" H 8100 1025 50  0001 L TNN
 F 4 "C13585" H 8000 1400 50  0001 C CNN "LCSC"
@@
 F 0 "D2" H 9200 1300 50  0000 L CNN
 F 1 "SK6812MINI-E" H 9294 1355 50  0001 L CNN
-F 2 "mycropad:LED_SK6812MINI-E_REV02_PLCC4_3.5x3.5mm_P1.75mm" H 9000 1100 50  0001 L TNN
+F 2 "mycropad:LED_SK6812MINI-E_REV02_PLCC4_3.5x3.5mm_P1.75mm___V2" H 9000 1100 50  0001 L TNN
 F 3 "https://cdn-shop.adafruit.com/product-files/4960/4960_SK6812MINI-E_REV02_EN.pdf" H 9050 1025 50  0001 L TNN
 	1    8950 1400
@@
 F 0 "D3" H 10150 1300 50  0000 L CNN
 F 1 "SK6812MINI-E" H 10244 1355 50  0001 L CNN
-F 2 "mycropad:LED_SK6812MINI-E_REV02_PLCC4_3.5x3.5mm_P1.75mm" H 9950 1100 50  0001 L TNN
+F 2 "mycropad:LED_SK6812MINI-E_REV02_PLCC4_3.5x3.5mm_P1.75mm___V2" H 9950 1100 50  0001 L TNN
 F 3 "https://cdn-shop.adafruit.com/product-files/4960/4960_SK6812MINI-E_REV02_EN.pdf" H 10000 1025 50  0001 L TNN
 	1    9900 1400
@@
 F 0 "D4" H 8250 2650 50  0000 L CNN
 F 1 "SK6812MINI-E" H 8344 2705 50  0001 L CNN
-F 2 "mycropad:LED_SK6812MINI-E_REV02_PLCC4_3.5x3.5mm_P1.75mm" H 8050 2450 50  0001 L TNN
+F 2 "mycropad:LED_SK6812MINI-E_REV02_PLCC4_3.5x3.5mm_P1.75mm___V2" H 8050 2450 50  0001 L TNN
 F 3 "https://cdn-shop.adafruit.com/product-files/4960/4960_SK6812MINI-E_REV02_EN.pdf" H 8100 2375 50  0001 L TNN
 	1    8000 2750
@@
 F 0 "D5" H 9200 2650 50  0000 L CNN
 F 1 "SK6812MINI-E" H 9294 2705 50  0001 L CNN
-F 2 "mycropad:LED_SK6812MINI-E_REV02_PLCC4_3.5x3.5mm_P1.75mm" H 9000 2450 50  0001 L TNN
+F 2 "mycropad:LED_SK6812MINI-E_REV02_PLCC4_3.5x3.5mm_P1.75mm___V2" H 9000 2450 50  0001 L TNN
 F 3 "https://cdn-shop.adafruit.com/product-files/4960/4960_SK6812MINI-E_REV02_EN.pdf" H 9050 2375 50  0001 L TNN
 	1    8950 2750
@@
 F 0 "D6" H 10150 2650 50  0000 L CNN
 F 1 "SK6812MINI-E" H 10244 2705 50  0001 L CNN
-F 2 "mycropad:LED_SK6812MINI-E_REV02_PLCC4_3.5x3.5mm_P1.75mm" H 9950 2450 50  0001 L TNN
+F 2 "mycropad:LED_SK6812MINI-E_REV02_PLCC4_3.5x3.5mm_P1.75mm___V2" H 9950 2450 50  0001 L TNN
 F 3 "https://cdn-shop.adafruit.com/product-files/4960/4960_SK6812MINI-E_REV02_EN.pdf" H 10000 2375 50  0001 L TNN
 	1    9900 2750
@@
 F 0 "D7" H 8250 4000 50  0000 L CNN
 F 1 "SK6812MINI-E" H 8344 4055 50  0001 L CNN
-F 2 "mycropad:LED_SK6812MINI-E_REV02_PLCC4_3.5x3.5mm_P1.75mm" H 8050 3800 50  0001 L TNN
+F 2 "mycropad:LED_SK6812MINI-E_REV02_PLCC4_3.5x3.5mm_P1.75mm___V2" H 8050 3800 50  0001 L TNN
 F 3 "https://cdn-shop.adafruit.com/product-files/4960/4960_SK6812MINI-E_REV02_EN.pdf" H 8100 3725 50  0001 L TNN
 	1    8000 4100
@@
 F 0 "D8" H 9200 4000 50  0000 L CNN
 F 1 "SK6812MINI-E" H 9294 4055 50  0001 L CNN
-F 2 "mycropad:LED_SK6812MINI-E_REV02_PLCC4_3.5x3.5mm_P1.75mm" H 9000 3800 50  0001 L TNN
+F 2 "mycropad:LED_SK6812MINI-E_REV02_PLCC4_3.5x3.5mm_P1.75mm___V2" H 9000 3800 50  0001 L TNN
 F 3 "https://cdn-shop.adafruit.com/product-files/4960/4960_SK6812MINI-E_REV02_EN.pdf" H 9050 3725 50  0001 L TNN
 	1    8950 4100
